File: hardware/name-blinker-2.sch (KiCad schematic (older format))
At the start: 48 parts, among them M1 MOUNTING-HOLE, M10 MOUNTING-HOLE, M12 MOUNTING-HOLE, M13 MOUNTING-HOLE, M2 MOUNTING-HOLE, M3 MOUNTING-HOLE, M4 MOUNTING-HOLE, M5 MOUNTING-HOLE, M6 MOUNTING-HOLE, M7 MOUNTING-HOLE, M8 MOUNTING-HOLE, M9 MOUNTING-HOLE, P2 USB_OTG, SW2 SMD-TOGGLE-SWITCH-2CH_2X3P-7X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, U1 MCP73831, U2 BMD-300, U3 TPS63051

Commit message: charging circuit side
Parts:
- P1: renamed from P?; footprint (none) -> Pin_Headers:Pin_Header_Angled_1x09
Connections:
- net +3V3: now also P1.7 (P7); no longer P1.3 (P3)
- net +5V: now also P1.9 (P9); no longer P1.1 (P1)
- net GND: now also P1.3 (P3), P1.6 (P6); no longer P1.4 (P4), P1.7 (P7)
- net SWCLK: now also P1.1 (P1); no longer P1.9 (P9)
- net SWDIO: now also P1.2 (P2); no longer P1.8 (P8)
- net UART_RX: now also P1.4 (P4); no longer P1.6 (P6)
- net VCC: now also P1.8 (P8); no longer P1.2 (P2)
Other:
- moved on the sheet: P1
Changed lines of the file:
@@
 L +5V #PWR04
 U 1 1 577B3A6B
-P 7400 900
-F 0 "#PWR04" H 7400 750 50  0001 C CNN
-F 1 "+5V" H 7400 1040 50  0000 C CNN
-F 2 "" H 7400 900 50  0000 C CNN
-F 3 "" H 7400 900 50  0000 C CNN
-	1    7400 900
+P 7300 950
+F 0 "#PWR04" H 7300 800 50  0001 C CNN
+F 1 "+5V" H 7300 1090 50  0000 C CNN
+F 2 "" H 7300 950 50  0000 C CNN
+F 3 "" H 7300 950 50  0000 C CNN
+	1    7300 950
 	1    0    0    -1
 $EndComp
@@
 L GND #PWR05
 U 1 1 577B3A85
-P 6950 2050
-F 0 "#PWR05" H 6950 1800 50  0001 C CNN
-F 1 "GND" H 6950 1900 50  0000 C CNN
-F 2 "" H 6950 2050 50  0000 C CNN
-F 3 "" H 6950 2050 50  0000 C CNN
-	1    6950 2050
+P 7850 1950
+F 0 "#PWR05" H 7850 1700 50  0001 C CNN
+F 1 "GND" H 7850 1800 50  0000 C CNN
+F 2 "" H 7850 1950 50  0000 C CNN
+F 3 "" H 7850 1950 50  0000 C CNN
+	1    7850 1950
 	1    0    0    -1
 $EndComp
@@
 Text GLabel 5000 1100 2    60   Input ~ 0
 SWCLK
-Text GLabel 7500 1700 0    60   Input ~ 0
+Text GLabel 7200 1750 2    60   Input ~ 0
 SWDIO
-Text GLabel 7500 1800 0    60   Input ~ 0
-SWCLK
-Text GLabel 7500 1400 0    60   Input ~ 0
+Text GLabel 7200 1450 2    60   Input ~ 0
 UART_TX
-Text GLabel 7500 1500 0    60   Input ~ 0
+Text GLabel 7200 1550 2    60   Input ~ 0
 UART_RX
 Text GLabel 3850 3150 3    60   Input ~ 0
@@
 	2450 1300 2950 1300
 Wire Wire Line
-	2450 700  2450 900
-Wire Wire Line
-	2450 900  2450 1000
-Wire Wire Line
-	2450 1000 2450 1100
-Wire Wire Line
-	2450 1100 2450 1200
-Wire Wire Line
-	2450 1200 2450 1300
-Wire Wire Line
-	2450 1300 2450 1350
+	2450 700  2450 1350
 Wire Wire Line
 	2950 1200 2450 1200
@@
 	4950 900  5550 900
 Wire Wire Line
-	5550 700  5550 900
-Wire Wire Line
-	5550 900  5550 1050
+	5550 700  5550 1050
 Wire Wire Line
 	4950 700  5550 700
@@
 	4950 1100 5000 1100
 Wire Wire Line
-	7650 1700 7500 1700
-Wire Wire Line
-	7650 1800 7500 1800
-Wire Wire Line
-	7650 1400 7500 1400
-Wire Wire Line
-	7650 1500 7500 1500
-Wire Wire Line
 	3350 3100 3350 3200
 Wire Wire Line
 	3350 3200 2750 3200
 Wire Wire Line
-	2750 3000 2750 3200
-Wire Wire Line
-	2750 3200 2750 3300
+	2750 3000 2750 3300
 Wire Wire Line
 	3850 3100 3850 3150
@@
 	4050 3100 4050 3150
 Wire Wire Line
-	8300 4400 8300 4750
-Wire Wire Line
-	8300 4750 8300 5050
-Wire Wire Line
-	8300 5350 8300 5550
-Wire Wire Line
-	8300 5550 8300 5650
-Wire Wire Line
-	7400 4750 7900 4750
-Wire Wire Line
-	7900 4750 8300 4750
-Wire Wire Line
-	8300 4750 8800 4750
+	8300 4400 8300 5050
+Wire Wire Line
+	8300 5350 8300 5650
+Wire Wire Line
+	7400 4750 8800 4750
 Wire Wire Line
 	7400 4950 7500 4950
@@
 	7500 4950 7500 5550
 Wire Wire Line
-	7500 5550 7650 5550
-Wire Wire Line
-	7650 5550 7900 5550
-Wire Wire Line
-	7900 5550 8300 5550
-Wire Wire Line
-	8300 5550 8800 5550
+	7500 5550 8800 5550
 Connection ~ 8300 5550
 Wire Wire Line
@@
 	10400 4650 10350 4650
 Wire Wire Line
-	10350 4650 10350 5450
-Wire Wire Line
 	10800 4850 10800 4950
 Wire Wire Line
 	10800 5250 10800 5350
-Wire Wire Line
-	10800 5350 10350 5350
-Wire Wire Line
-	10350 5350 10350 5400
 Wire Wire Line
 	7900 5100 7900 4750
@@
 	5850 5200 5850 5350
 Wire Wire Line
-	5850 4600 5850 4750
-Wire Wire Line
-	5850 4750 5850 4900
+	5850 4600 5850 4900
 Connection ~ 5850 4750
 Wire Wire Line
@@
 	6250 5200 6250 5100
 Wire Wire Line
-	6250 5600 6250 5700
-Wire Wire Line
-	6250 5700 6250 5850
+	6250 5600 6250 5850
 Wire Wire Line
 	6250 6250 6250 6150
@@
 	8800 5550 8800 5350
 Wire Wire Line
-	5850 4750 6250 4750
-Wire Wire Line
-	6250 4750 6600 4750
+	5850 4750 6600 4750
 Wire Wire Line
 	6450 5700 6250 5700
@@
 	4350 4200 4350 4100
 Wire Wire Line
-	7650 1000 7400 1000
-Wire Wire Line
-	7400 1000 7400 900
-Wire Wire Line
-	7050 1200 7650 1200
-Wire Wire Line
-	7050 1200 7050 1100
+	7300 1050 7300 950
+Wire Wire Line
+	7600 1250 7600 1150
 $Comp
 L MOUNTING-HOLE M12
@@
 	4250 3650 4250 3100
 Wire Wire Line
-	2750 4300 3150 4300
-Wire Wire Line
-	3150 4300 3250 4300
-Wire Wire Line
-	3250 4300 3450 4300
-Wire Wire Line
-	3450 4300 4550 4300
-Wire Wire Line
-	4550 4300 4750 4300
+	2750 4300 4750 4300
 Wire Wire Line
 	3250 4300 3250 4350
@@
 L +3.3V #PWR016
 U 1 1 57811A79
-P 7050 1100
-F 0 "#PWR016" H 7050 950 50  0001 C CNN
-F 1 "+3.3V" H 7050 1240 50  0000 C CNN
-F 2 "" H 7050 1100 50  0000 C CNN
-F 3 "" H 7050 1100 50  0000 C CNN
-	1    7050 1100
+P 7600 1150
+F 0 "#PWR016" H 7600 1000 50  0001 C CNN
+F 1 "+3.3V" H 7600 1290 50  0000 C CNN
+F 2 "" H 7600 1150 50  0000 C CNN
+F 3 "" H 7600 1150 50  0000 C CNN
+	1    7600 1150
 	1    0    0    -1
 $EndComp
@@
 	2300 5550 2300 5100
 Wire Wire Line
-	1650 5100 2300 5100
-Wire Wire Line
-	2300 5100 2500 5100
-Wire Wire Line
-	2500 5100 3300 5100
-Wire Wire Line
-	1650 5000 1650 5100
-Wire Wire Line
-	1650 5100 1650 5200
-Wire Wire Line
-	1650 5500 1650 5550
-Wire Wire Line
-	1650 5550 1650 5600
+	1650 5100 3300 5100
+Wire Wire Line
+	1650 5000 1650 5200
+Wire Wire Line
+	1650 5500 1650 5600
 $Comp
 L VCC #PWR018
@@
 	1700 6450 1450 6450
 Wire Wire Line
-	1450 6450 1450 6800
-Wire Wire Line
-	1450 6800 1450 6850
-Wire Wire Line
-	1450 6850 1450 7050
-Wire Wire Line
-	1450 7050 1450 7300
-Wire Wire Line
-	1450 7300 1450 7500
+	1450 6450 1450 7500
 Wire Wire Line
 	1500 6850 1450 6850
@@
 	1800 7050 2050 7050
 Wire Wire Line
-	2050 7050 2050 7300
-Wire Wire Line
-	2050 7300 2050 7350
-Wire Wire Line
-	1800 7300 2050 7300
-Wire Wire Line
-	2050 7300 2500 7300
+	2050 7050 2050 7350
+Wire Wire Line
+	1800 7300 2500 7300
 Connection ~ 2050 7300
 Wire Wire Line
@@
 $EndComp
 Wire Wire Line
-	1950 1900 1950 2000
-Wire Wire Line
-	1950 2000 1950 2100
+	1950 1900 1950 2100
 Connection ~ 1950 2000
 Wire Wire Line
@@
 L VCC #PWR025
 U 1 1 578150D2
-P 7250 950
-F 0 "#PWR025" H 7250 800 50  0001 C CNN
-F 1 "VCC" H 7250 1100 50  0000 C CNN
-F 2 "" H 7250 950 50  0000 C CNN
-F 3 "" H 7250 950 50  0000 C CNN
-	1    7250 950
-	1    0    0    -1
-$EndComp
-Wire Wire Line
-	7250 950  7250 1100
-Wire Wire Line
-	7250 1100 7650 1100
-Wire Wire Line
-	7650 1300 6950 1300
-Wire Wire Line
-	6950 1300 6950 1600
-Wire Wire Line
-	6950 1600 6950 1900
-Wire Wire Line
-	6950 1900 6950 2050
-Wire Wire Line
-	7650 1600 6950 1600
-Connection ~ 6950 1600
-$Comp
-L CONN_01X09 P?
+P 7450 1000
+F 0 "#PWR025" H 7450 850 50  0001 C CNN
+F 1 "VCC" H 7450 1150 50  0000 C CNN
+F 2 "" H 7450 1000 50  0000 C CNN
+F 3 "" H 7450 1000 50  0000 C CNN
+	1    7450 1000
+	1    0    0    -1
+$EndComp
+Wire Wire Line
+	7450 1000 7450 1150
+$Comp
+L CONN_01X09 P1
 U 1 1 57815D7E
-P 7850 1400
-F 0 "P?" H 7850 1900 50  0000 C CNN
-F 1 "CONN_01X09" V 7950 1400 50  0000 C CNN
-F 2 "" H 7850 1400 50  0000 C CNN
-F 3 "" H 7850 1400 50  0000 C CNN
-	1    7850 1400
-	1    0    0    -1
-$EndComp
+P 6900 1450
+F 0 "P1" H 6900 1950 50  0000 C CNN
+F 1 "CONN_01X09" V 7000 1450 50  0000 C CNN
+F 2 "Pin_Headers:Pin_Header_Angled_1x09" H 6900 1450 50  0001 C CNN
+F 3 "" H 6900 1450 50  0000 C CNN
+	1    6900 1450
+	-1   0    0    1
+$EndComp
+Wire Wire Line
+	7100 1050 7300 1050
+Wire Wire Line
+	7450 1150 7100 1150
+Wire Wire Line
+	7100 1250 7600 1250
+Text GLabel 7200 1850 2    60   Input ~ 0
+SWCLK
+Wire Wire Line
+	7100 1450 7200 1450
+Wire Wire Line
+	7100 1550 7200 1550
+Wire Wire Line
+	7100 1750 7200 1750
+Wire Wire Line
+	7100 1850 7200 1850
+Wire Wire Line
+	7100 1650 7850 1650
+Wire Wire Line
+	7850 1350 7850 1950
+Wire Wire Line
+	7100 1350 7850 1350
+Connection ~ 7850 1650
+Wire Wire Line
+	10350 4650 10350 5450
+Wire Wire Line
+	10800 5350 10350 5350
+Connection ~ 10350 5350
 $EndSCHEMATC

Commit message: connected all wires
Parts:
- removed C4, C5: 330pF, Capacitors_SMD:C_0805_HandSoldering, symbol C
- added M11: MOUNTING-HOLE, Mounting_Holes:MountingHole_2.5mm_Pad, symbol MOUNTING-HOLE
- BT2: footprint Connectors_Molex:Molex_MicroLatch-53254-0270_02x2.00mm_Angled -> jst:Molex_MicroLatch-53254-0270_02x2.00mm_Angled
Connections:
- net GND: now also M11.1
- net In0: now also U2.P9 (P0.28/AIN4); no longer U2.P23 (P0.07)
- net at U2.P11 (P0.30/AIN6): now also R14.2, R15.1
- now unconnected: U2.P12 (P0.31/AIN7)
Other:
- moved on the sheet: R14, R15
Changed lines of the file:
@@
 F 0 "BT2" H 8900 5250 50  0000 L CNN
 F 1 "JST" H 8900 5150 50  0000 L CNN
-F 2 "Connectors_Molex:Molex_MicroLatch-53254-0270_02x2.00mm_Angled" V 8800 5240 50  0001 C CNN
+F 2 "jst:Molex_MicroLatch-53254-0270_02x2.00mm_Angled" V 8800 5240 50  0001 C CNN
 F 3 "" V 8800 5240 50  0000 C CNN
 	1    8800 5200
@@
 L MOUNTING-HOLE M1
 U 1 1 577BA5E6
-P 10950 750
-F 0 "M1" H 11050 750 40  0001 C CNN
-F 1 "MOUNTING-HOLE" H 10950 650 40  0001 C CNN
-F 2 "Mounting_Holes:MountingHole_2.5mm_Pad" H 10950 500 60  0001 C CNN
-F 3 "" H 10950 500 60  0000 C CNN
-	1    10950 750
-	1    0    0    -1
-$EndComp
-Text GLabel 10100 750  0    60   Input ~ 0
+P 10950 650
+F 0 "M1" H 11050 650 40  0001 C CNN
+F 1 "MOUNTING-HOLE" H 10950 550 40  0001 C CNN
+F 2 "Mounting_Holes:MountingHole_2.5mm_Pad" H 10950 400 60  0001 C CNN
+F 3 "" H 10950 400 60  0000 C CNN
+	1    10950 650
+	1    0    0    -1
+$EndComp
+Text GLabel 10100 650  0    60   Input ~ 0
 In0
 Wire Wire Line
-	10100 750  10950 750
-Text GLabel 3950 3600 3    60   Input ~ 0
+	10100 650  10950 650
+Text GLabel 2700 1700 0    60   Input ~ 0
 In0
-Wire Wire Line
-	3950 3600 3950 3100
 $Comp
 L SMD-TOGGLE-SWITCH-2CH_2X3P-7X3.5MM_ SW2
@@
 Wire Wire Line
 	8400 4400 8300 4400
-$Comp
-L C C4
-U 1 1 577BDD23
-P 4050 3950
-F 0 "C4" H 4075 4050 50  0000 L CNN
-F 1 "330pF" H 3800 3850 50  0000 L CNN
-F 2 "Capacitors_SMD:C_0805_HandSoldering" H 4088 3800 50  0001 C CNN
-F 3 "" H 4050 3950 50  0000 C CNN
-	1    4050 3950
-	1    0    0    -1
-$EndComp
-$Comp
-L C C5
-U 1 1 577BDD97
-P 4350 3950
-F 0 "C5" H 4375 4050 50  0000 L CNN
-F 1 "330pF" H 4100 3850 50  0000 L CNN
-F 2 "Capacitors_SMD:C_0805_HandSoldering" H 4388 3800 50  0001 C CNN
-F 3 "" H 4350 3950 50  0000 C CNN
-	1    4350 3950
-	1    0    0    -1
-$EndComp
-Wire Wire Line
-	4250 3650 4350 3650
-Wire Wire Line
-	4350 3650 4350 3800
-Wire Wire Line
-	4150 3650 4050 3650
-Wire Wire Line
-	4050 3650 4050 3800
-Wire Wire Line
-	4050 4100 4050 4200
-Wire Wire Line
-	4050 4200 4350 4200
-Wire Wire Line
-	4350 4200 4350 4100
 Wire Wire Line
 	7300 1050 7300 950
@@
 L MOUNTING-HOLE M12
 U 1 1 577B70EB
-P 10950 1150
-F 0 "M12" H 11050 1150 40  0001 C CNN
-F 1 "MOUNTING-HOLE" H 10950 1050 40  0001 C CNN
-F 2 "Mounting_Holes:MountingHole_2.5mm_Pad" H 10950 900 60  0001 C CNN
-F 3 "" H 10950 900 60  0000 C CNN
-	1    10950 1150
-	1    0    0    -1
-$EndComp
-Wire Wire Line
-	10050 1150 10950 1150
+P 10950 1250
+F 0 "M12" H 11050 1250 40  0001 C CNN
+F 1 "MOUNTING-HOLE" H 10950 1150 40  0001 C CNN
+F 2 "Mounting_Holes:MountingHole_2.5mm_Pad" H 10950 1000 60  0001 C CNN
+F 3 "" H 10950 1000 60  0000 C CNN
+	1    10950 1250
+	1    0    0    -1
+$EndComp
+Wire Wire Line
+	10050 1250 10950 1250
 $Comp
 L MOUNTING-HOLE M13
 U 1 1 577B86A7
-P 10950 950
-F 0 "M13" H 11050 950 40  0001 C CNN
-F 1 "MOUNTING-HOLE" H 10950 850 40  0001 C CNN
-F 2 "Mounting_Holes:MountingHole_2.5mm_Pad" H 10950 700 60  0001 C CNN
-F 3 "" H 10950 700 60  0000 C CNN
-	1    10950 950
+P 10950 850
+F 0 "M13" H 11050 850 40  0001 C CNN
+F 1 "MOUNTING-HOLE" H 10950 750 40  0001 C CNN
+F 2 "Mounting_Holes:MountingHole_2.5mm_Pad" H 10950 600 60  0001 C CNN
+F 3 "" H 10950 600 60  0000 C CNN
+	1    10950 850
 	1    0    0    -1
 $EndComp
@@
 L GND #PWR013
 U 1 1 577B86AD
-P 10050 950
-F 0 "#PWR013" H 10050 700 50  0001 C CNN
-F 1 "GND" H 10050 800 50  0000 C CNN
-F 2 "" H 10050 950 50  0000 C CNN
-F 3 "" H 10050 950 50  0000 C CNN
-	1    10050 950
-	0    1    1    0
-$EndComp
-Wire Wire Line
-	10050 950  10950 950
+P 10050 850
+F 0 "#PWR013" H 10050 600 50  0001 C CNN
+F 1 "GND" H 10050 700 50  0000 C CNN
+F 2 "" H 10050 850 50  0000 C CNN
+F 3 "" H 10050 850 50  0000 C CNN
+	1    10050 850
+	0    1    1    0
+$EndComp
+Wire Wire Line
+	10050 850  10950 850
 $Comp
 L C C6
@@
 $EndComp
 Wire Wire Line
-	4150 3650 4150 3100
-Wire Wire Line
-	4250 3650 4250 3100
-Wire Wire Line
 	2750 4300 4750 4300
 Wire Wire Line
@@
 L +3.3V #PWR015
 U 1 1 578115B5
-P 10050 1150
-F 0 "#PWR015" H 10050 1000 50  0001 C CNN
-F 1 "+3.3V" H 10050 1290 50  0000 C CNN
-F 2 "" H 10050 1150 50  0000 C CNN
-F 3 "" H 10050 1150 50  0000 C CNN
-	1    10050 1150
+P 10050 1250
+F 0 "#PWR015" H 10050 1100 50  0001 C CNN
+F 1 "+3.3V" H 10050 1390 50  0000 C CNN
+F 2 "" H 10050 1250 50  0000 C CNN
+F 3 "" H 10050 1250 50  0000 C CNN
+	1    10050 1250
 	0    -1   -1   0
 $EndComp
@@
 L VCC #PWR023
 U 1 1 5783A258
-P 1950 1450
-F 0 "#PWR023" H 1950 1300 50  0001 C CNN
-F 1 "VCC" H 1950 1600 50  0000 C CNN
-F 2 "" H 1950 1450 50  0000 C CNN
-F 3 "" H 1950 1450 50  0000 C CNN
-	1    1950 1450
+P 1950 1350
+F 0 "#PWR023" H 1950 1200 50  0001 C CNN
+F 1 "VCC" H 1950 1500 50  0000 C CNN
+F 2 "" H 1950 1350 50  0000 C CNN
+F 3 "" H 1950 1350 50  0000 C CNN
+	1    1950 1350
 	1    0    0    -1
 $EndComp
@@
 L GND #PWR024
 U 1 1 5783A2B0
-P 1950 2500
-F 0 "#PWR024" H 1950 2250 50  0001 C CNN
-F 1 "GND" H 1950 2350 50  0000 C CNN
-F 2 "" H 1950 2500 50  0000 C CNN
-F 3 "" H 1950 2500 50  0000 C CNN
-	1    1950 2500
+P 1950 2400
+F 0 "#PWR024" H 1950 2150 50  0001 C CNN
+F 1 "GND" H 1950 2250 50  0000 C CNN
+F 2 "" H 1950 2400 50  0000 C CNN
+F 3 "" H 1950 2400 50  0000 C CNN
+	1    1950 2400
 	1    0    0    -1
 $EndComp
@@
 L R R14
 U 1 1 5783A69E
-P 1950 1750
-F 0 "R14" V 2030 1750 50  0000 C CNN
-F 1 "800K" V 1950 1750 50  0000 C CNN
-F 2 "Resistors_SMD:R_0805_HandSoldering" V 1880 1750 50  0001 C CNN
-F 3 "" H 1950 1750 50  0000 C CNN
-	1    1950 1750
+P 1950 1650
+F 0 "R14" V 2030 1650 50  0000 C CNN
+F 1 "800K" V 1950 1650 50  0000 C CNN
+F 2 "Resistors_SMD:R_0805_HandSoldering" V 1880 1650 50  0001 C CNN
+F 3 "" H 1950 1650 50  0000 C CNN
+	1    1950 1650
 	1    0    0    -1
 $EndComp
@@
 L R R15
 U 1 1 5783A73F
-P 1950 2250
-F 0 "R15" V 2030 2250 50  0000 C CNN
-F 1 "2M" V 1950 2250 50  0000 C CNN
-F 2 "Resistors_SMD:R_0805_HandSoldering" V 1880 2250 50  0001 C CNN
-F 3 "" H 1950 2250 50  0000 C CNN
-	1    1950 2250
-	1    0    0    -1
-$EndComp
-Wire Wire Line
-	1950 1900 1950 2100
-Connection ~ 1950 2000
-Wire Wire Line
-	1950 1600 1950 1450
-Wire Wire Line
-	1950 2500 1950 2400
-Wire Wire Line
-	2950 2000 1950 2000
+P 1950 2150
+F 0 "R15" V 2030 2150 50  0000 C CNN
+F 1 "2M" V 1950 2150 50  0000 C CNN
+F 2 "Resistors_SMD:R_0805_HandSoldering" V 1880 2150 50  0001 C CNN
+F 3 "" H 1950 2150 50  0000 C CNN
+	1    1950 2150
+	1    0    0    -1
+$EndComp
+Wire Wire Line
+	1950 1800 1950 2000
+Wire Wire Line
+	1950 1500 1950 1350
+Wire Wire Line
+	1950 2400 1950 2300
 $Comp
 L LPS3015 L1
@@
 	10800 5350 10350 5350
 Connection ~ 10350 5350
+$Comp
+L MOUNTING-HOLE M11
+U 1 1 5781CFF7
+P 10950 1050
+F 0 "M11" H 11050 1050 40  0001 C CNN
+F 1 "MOUNTING-HOLE" H 10950 950 40  0001 C CNN
+F 2 "Mounting_Holes:MountingHole_2.5mm_Pad" H 10950 800 60  0001 C CNN
+F 3 "" H 10950 800 60  0000 C CNN
+	1    10950 1050
+	1    0    0    -1
+$EndComp
+$Comp
+L GND #PWR026
+U 1 1 5781CFFD
+P 10050 1050
+F 0 "#PWR026" H 10050 800 50  0001 C CNN
+F 1 "GND" H 10050 900 50  0000 C CNN
+F 2 "" H 10050 1050 50  0000 C CNN
+F 3 "" H 10050 1050 50  0000 C CNN
+	1    10050 1050
+	0    1    1    0
+$EndComp
+Wire Wire Line
+	10050 1050 10950 1050
+Wire Wire Line
+	2700 1700 2950 1700
+Wire Wire Line
+	2950 1900 1950 1900
+Connection ~ 1950 1900
 $EndSCHEMATC

Commit message: connected everything
Parts:
- added D? (x9): LED, symbol LED
- added SW?: SW_PUSH, symbol SW_PUSH
Connections:
- net GND: now also D?.1 (K), D?.1 (K), D?.1 (K), D?.1 (K), D?.1 (K), D?.1 (K), D?.1 (K), D?.1 (K), D?.1 (K), SW?.2; no longer D2.1 (K)
- net In0: now also SW?.1
- net at M2.1, R1.1: now also D?.2 (A)
- net at M3.1, R2.1: now also D?.2 (A)
- net at M4.1, R3.1: now also D?.2 (A)
- net at M5.1, R4.1: now also D?.2 (A)
- net at M6.1, R5.1: now also D?.2 (A)
- net at M7.1, R6.1: now also D?.2 (A)
- net at M8.1, R7.1: now also D?.2 (A)
- net at M9.1, R8.1: now also D?.2 (A)
- net at M10.1, R9.1: now also D?.2 (A)
Other:
- moved on the sheet: BT1, BT2, C1, C2, C3, D1, D2, P2, R1, R10, R11, R12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
