File: hardware/name-blinker-2.sch (KiCad schematic (older format))
At the start: 57 parts, among them M1 MOUNTING-HOLE, M10 MOUNTING-HOLE, M11 MOUNTING-HOLE, M12 MOUNTING-HOLE, M13 MOUNTING-HOLE, M2 MOUNTING-HOLE, M3 MOUNTING-HOLE, M4 MOUNTING-HOLE, M5 MOUNTING-HOLE, M6 MOUNTING-HOLE, M7 MOUNTING-HOLE, M8 MOUNTING-HOLE, M9 MOUNTING-HOLE, P1 CONN_01X09, P2 USB_OTG, SW2 SMD-TOGGLE-SWITCH-2CH_2X3P-7X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, U1 MCP73831, U2 BMD-300, U3 TPS63051

Commit message: silkscreen stuff
Parts:
- removed M11: MOUNTING-HOLE, Mounting_Holes:MountingHole_2.5mm_Pad, symbol MOUNTING-HOLE
- D10, D11, D3, D4, D5, D6, D7, D8, D9: renamed from D?; footprint (none) -> LEDs:LED_0805
- SW1: renamed from SW?; footprint (none) -> Buttons_Switches_SMD:SW_SPST_B3S-1000
Changed lines of the file:
@@
 L MOUNTING-HOLE M13
 U 1 1 577B86A7
-P 10950 700
-F 0 "M13" H 11050 700 40  0001 C CNN
-F 1 "MOUNTING-HOLE" H 10950 600 40  0001 C CNN
-F 2 "Mounting_Holes:MountingHole_2.5mm_Pad" H 10950 450 60  0001 C CNN
-F 3 "" H 10950 450 60  0000 C CNN
-	1    10950 700
+P 10950 900
+F 0 "M13" H 11050 900 40  0001 C CNN
+F 1 "MOUNTING-HOLE" H 10950 800 40  0001 C CNN
+F 2 "Mounting_Holes:MountingHole_2.5mm_Pad" H 10950 650 60  0001 C CNN
+F 3 "" H 10950 650 60  0000 C CNN
+	1    10950 900
 	1    0    0    -1
 $EndComp
@@
 L GND #PWR013
 U 1 1 577B86AD
-P 10050 700
-F 0 "#PWR013" H 10050 450 50  0001 C CNN
-F 1 "GND" H 10050 550 50  0000 C CNN
-F 2 "" H 10050 700 50  0000 C CNN
-F 3 "" H 10050 700 50  0000 C CNN
-	1    10050 700
+P 10050 900
+F 0 "#PWR013" H 10050 650 50  0001 C CNN
+F 1 "GND" H 10050 750 50  0000 C CNN
+F 2 "" H 10050 900 50  0000 C CNN
+F 3 "" H 10050 900 50  0000 C CNN
+	1    10050 900
 	0    1    1    0
 $EndComp
 Wire Wire Line
-	10050 700  10950 700
+	10050 900  10950 900
 $Comp
 L C C6
@@
 	10700 6100 10250 6100
 Connection ~ 10250 6100
-$Comp
-L MOUNTING-HOLE M11
-U 1 1 5781CFF7
-P 10950 900
-F 0 "M11" H 11050 900 40  0001 C CNN
-F 1 "MOUNTING-HOLE" H 10950 800 40  0001 C CNN
-F 2 "Mounting_Holes:MountingHole_2.5mm_Pad" H 10950 650 60  0001 C CNN
-F 3 "" H 10950 650 60  0000 C CNN
-	1    10950 900
-	1    0    0    -1
-$EndComp
-$Comp
-L GND #PWR026
-U 1 1 5781CFFD
-P 10050 900
-F 0 "#PWR026" H 10050 650 50  0001 C CNN
-F 1 "GND" H 10050 750 50  0000 C CNN
-F 2 "" H 10050 900 50  0000 C CNN
-F 3 "" H 10050 900 50  0000 C CNN
-	1    10050 900
-	0    1    1    0
-$EndComp
-Wire Wire Line
-	10050 900  10950 900
 Wire Wire Line
 	2700 1700 2950 1700
@@
 Connection ~ 1950 1900
 $Comp
-L SW_PUSH SW?
+L SW_PUSH SW1
 U 1 1 5781F948
 P 10600 1500
-F 0 "SW?" H 10750 1610 50  0000 C CNN
+F 0 "SW1" H 10750 1610 50  0000 C CNN
 F 1 "SW_PUSH" H 10600 1420 50  0000 C CNN
-F 2 "" H 10600 1500 50  0000 C CNN
+F 2 "Buttons_Switches_SMD:SW_SPST_B3S-1000" H 10600 1500 50  0001 C CNN
 F 3 "" H 10600 1500 50  0000 C CNN
 	1    10600 1500
@@
 $EndComp
 $Comp
-L GND #PWR?
+L GND #PWR027
 U 1 1 5781F9CB
 P 11000 1500
-F 0 "#PWR?" H 11000 1250 50  0001 C CNN
+F 0 "#PWR027" H 11000 1250 50  0001 C CNN
 F 1 "GND" H 11000 1350 50  0000 C CNN
 F 2 "" H 11000 1500 50  0000 C CNN
@@
 Connection ~ 10150 1500
 $Comp
-L LED D?
+L LED D3
 U 1 1 5781FD4D
 P 10600 1900
-F 0 "D?" H 10600 2000 50  0000 C CNN
+F 0 "D3" H 10600 2000 50  0000 C CNN
 F 1 "LED" H 10600 1800 50  0000 C CNN
-F 2 "" H 10600 1900 50  0000 C CNN
+F 2 "LEDs:LED_0805" H 10600 1900 50  0001 C CNN
 F 3 "" H 10600 1900 50  0000 C CNN
 	1    10600 1900
@@
 $EndComp
 $Comp
-L GND #PWR?
+L GND #PWR028
 U 1 1 5781FDD2
 P 11000 1900
-F 0 "#PWR?" H 11000 1650 50  0001 C CNN
+F 0 "#PWR028" H 11000 1650 50  0001 C CNN
 F 1 "GND" H 11000 1750 50  0000 C CNN
 F 2 "" H 11000 1900 50  0000 C CNN
@@
 Connection ~ 10150 1900
 $Comp
-L LED D?
+L LED D4
 U 1 1 57820770
 P 10600 2200
-F 0 "D?" H 10600 2300 50  0000 C CNN
+F 0 "D4" H 10600 2300 50  0000 C CNN
 F 1 "LED" H 10600 2100 50  0000 C CNN
-F 2 "" H 10600 2200 50  0000 C CNN
+F 2 "LEDs:LED_0805" H 10600 2200 50  0001 C CNN
 F 3 "" H 10600 2200 50  0000 C CNN
 	1    10600 2200
@@
 $EndComp
 $Comp
-L LED D?
+L LED D5
 U 1 1 57821B8A
 P 10600 2500
-F 0 "D?" H 10600 2600 50  0000 C CNN
+F 0 "D5" H 10600 2600 50  0000 C CNN
 F 1 "LED" H 10600 2400 50  0000 C CNN
-F 2 "" H 10600 2500 50  0000 C CNN
+F 2 "LEDs:LED_0805" H 10600 2500 50  0001 C CNN
 F 3 "" H 10600 2500 50  0000 C CNN
 	1    10600 2500
@@
 $EndComp
 $Comp
-L LED D?
+L LED D6
 U 1 1 57821C18
 P 10600 2800
-F 0 "D?" H 10600 2900 50  0000 C CNN
+F 0 "D6" H 10600 2900 50  0000 C CNN
 F 1 "LED" H 10600 2700 50  0000 C CNN
-F 2 "" H 10600 2800 50  0000 C CNN
+F 2 "LEDs:LED_0805" H 10600 2800 50  0001 C CNN
 F 3 "" H 10600 2800 50  0000 C CNN
 	1    10600 2800
@@
 $EndComp
 $Comp
-L LED D?
+L LED D7
 U 1 1 57821CAB
 P 10600 3100
-F 0 "D?" H 10600 3200 50  0000 C CNN
+F 0 "D7" H 10600 3200 50  0000 C CNN
 F 1 "LED" H 10600 3000 50  0000 C CNN
-F 2 "" H 10600 3100 50  0000 C CNN
+F 2 "LEDs:LED_0805" H 10600 3100 50  0001 C CNN
 F 3 "" H 10600 3100 50  0000 C CNN
 	1    10600 3100
@@
 $EndComp
 $Comp
-L LED D?
+L LED D8
 U 1 1 57821E17
 P 10600 3400
-F 0 "D?" H 10600 3500 50  0000 C CNN
+F 0 "D8" H 10600 3500 50  0000 C CNN
 F 1 "LED" H 10600 3300 50  0000 C CNN
-F 2 "" H 10600 3400 50  0000 C CNN
+F 2 "LEDs:LED_0805" H 10600 3400 50  0001 C CNN
 F 3 "" H 10600 3400 50  0000 C CNN
 	1    10600 3400
@@
 $EndComp
 $Comp
-L LED D?
+L LED D9
 U 1 1 57821F9A
 P 10600 3700
-F 0 "D?" H 10600 3800 50  0000 C CNN
+F 0 "D9" H 10600 3800 50  0000 C CNN
 F 1 "LED" H 10600 3600 50  0000 C CNN
-F 2 "" H 10600 3700 50  0000 C CNN
+F 2 "LEDs:LED_0805" H 10600 3700 50  0001 C CNN
 F 3 "" H 10600 3700 50  0000 C CNN
 	1    10600 3700
@@
 $EndComp
 $Comp
-L LED D?
+L LED D10
 U 1 1 5782203A
 P 10600 4000
-F 0 "D?" H 10600 4100 50  0000 C CNN
+F 0 "D10" H 10600 4100 50  0000 C CNN
 F 1 "LED" H 10600 3900 50  0000 C CNN
-F 2 "" H 10600 4000 50  0000 C CNN
+F 2 "LEDs:LED_0805" H 10600 4000 50  0001 C CNN
 F 3 "" H 10600 4000 50  0000 C CNN
 	1    10600 4000
@@
 $EndComp
 $Comp
-L LED D?
+L LED D11
 U 1 1 578220D7
 P 10600 4300
-F 0 "D?" H 10600 4400 50  0000 C CNN
+F 0 "D11" H 10600 4400 50  0000 C CNN
 F 1 "LED" H 10600 4200 50  0000 C CNN
-F 2 "" H 10600 4300 50  0000 C CNN
+F 2 "LEDs:LED_0805" H 10600 4300 50  0001 C CNN
 F 3 "" H 10600 4300 50  0000 C CNN
 	1    10600 4300
@@
 $EndComp
 $Comp
-L GND #PWR?
+L GND #PWR029
 U 1 1 5782227B
 P 11000 2200
-F 0 "#PWR?" H 11000 1950 50  0001 C CNN
+F 0 "#PWR029" H 11000 1950 50  0001 C CNN
 F 1 "GND" H 11000 2050 50  0000 C CNN
 F 2 "" H 11000 2200 50  0000 C CNN
@@
 $EndComp
 $Comp
-L GND #PWR?
+L GND #PWR030
 U 1 1 578222D9
 P 11000 2500
-F 0 "#PWR?" H 11000 2250 50  0001 C CNN
+F 0 "#PWR030" H 11000 2250 50  0001 C CNN
 F 1 "GND" H 11000 2350 50  0000 C CNN
 F 2 "" H 11000 2500 50  0000 C CNN
@@
 $EndComp
 $Comp
-L GND #PWR?
+L GND #PWR031
 U 1 1 578222DF
 P 11000 2800
-F 0 "#PWR?" H 11000 2550 50  0001 C CNN
+F 0 "#PWR031" H 11000 2550 50  0001 C CNN
 F 1 "GND" H 11000 2650 50  0000 C CNN
 F 2 "" H 11000 2800 50  0000 C CNN
@@
 $EndComp
 $Comp
-L GND #PWR?
+L GND #PWR032
 U 1 1 5782233D
 P 11000 3100
-F 0 "#PWR?" H 11000 2850 50  0001 C CNN
+F 0 "#PWR032" H 11000 2850 50  0001 C CNN
 F 1 "GND" H 11000 2950 50  0000 C CNN
 F 2 "" H 11000 3100 50  0000 C CNN
@@
 $EndComp
 $Comp
-L GND #PWR?
+L GND #PWR033
 U 1 1 57822343
 P 11000 3400
-F 0 "#PWR?" H 11000 3150 50  0001 C CNN
+F 0 "#PWR033" H 11000 3150 50  0001 C CNN
 F 1 "GND" H 11000 3250 50  0000 C CNN
 F 2 "" H 11000 3400 50  0000 C CNN
@@
 $EndComp
 $Comp
-L GND #PWR?
+L GND #PWR034
 U 1 1 57822349
 P 11000 3700
-F 0 "#PWR?" H 11000 3450 50  0001 C CNN
+F 0 "#PWR034" H 11000 3450 50  0001 C CNN
 F 1 "GND" H 11000 3550 50  0000 C CNN
 F 2 "" H 11000 3700 50  0000 C CNN
@@
 $EndComp
 $Comp
-L GND #PWR?
+L GND #PWR035
 U 1 1 5782234F
 P 11000 4000
-F 0 "#PWR?" H 11000 3750 50  0001 C CNN
+F 0 "#PWR035" H 11000 3750 50  0001 C CNN
 F 1 "GND" H 11000 3850 50  0000 C CNN
 F 2 "" H 11000 4000 50  0000 C CNN
@@
 $EndComp
 $Comp
-L GND #PWR?
+L GND #PWR036
 U 1 1 578223AD
 P 11000 4300
-F 0 "#PWR?" H 11000 4050 50  0001 C CNN
+F 0 "#PWR036" H 11000 4050 50  0001 C CNN
 F 1 "GND" H 11000 4150 50  0000 C CNN
 F 2 "" H 11000 4300 50  0000 C CNN
