File: hardware/name-blinker-2.sch (KiCad schematic (older format))
At the start: 56 parts, among them M1 MOUNTING-HOLE, M10 MOUNTING-HOLE, M12 MOUNTING-HOLE, M13 MOUNTING-HOLE, M2 MOUNTING-HOLE, M3 MOUNTING-HOLE, M4 MOUNTING-HOLE, M5 MOUNTING-HOLE, M6 MOUNTING-HOLE, M7 MOUNTING-HOLE, M8 MOUNTING-HOLE, M9 MOUNTING-HOLE, P1 CONN_01X09, P2 USB_OTG, SW1 SW_PUSH, SW2 SMD-TOGGLE-SWITCH-2CH_2X3P-7X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, U1 MCP73831, U2 BMD-300, U3 TPS63051

Commit message: change mounting hole reference name to be in line with connected NRF pins
Parts:
- renumbered M13 to M0, M6 to M11, M7 to M12, M8 to M13, M9 to M17, M10 to M19, M1 to M28, M12 to M33
Changed lines of the file:
@@
 Sheet 1 1
 Title "Name Blinker 2"
-Date "2016-07-10"
+Date "2016-07-22"
 Rev "1"
 Comp ""
@@
 U 1 1 577B965C
 P 10150 1900
-F 0 "M2" H 10250 1900 40  0001 C CNN
+F 0 "M2" H 10150 2000 40  0000 C CNN
 F 1 "MOUNTING-HOLE" H 10150 1800 40  0001 C CNN
 F 2 "Mounting_Holes:MountingHole_2.5mm_Pad" H 10150 1650 60  0001 C CNN
@@
 U 1 1 577B9A0D
 P 10150 2200
-F 0 "M3" H 10250 2200 40  0001 C CNN
+F 0 "M3" H 10150 2300 40  0000 C CNN
 F 1 "MOUNTING-HOLE" H 10150 2100 40  0001 C CNN
 F 2 "Mounting_Holes:MountingHole_2.5mm_Pad" H 10150 1950 60  0001 C CNN
@@
 U 1 1 577B9AAE
 P 10150 2500
-F 0 "M4" H 10250 2500 40  0001 C CNN
+F 0 "M4" H 10150 2600 40  0000 C CNN
 F 1 "MOUNTING-HOLE" H 10150 2400 40  0001 C CNN
 F 2 "Mounting_Holes:MountingHole_2.5mm_Pad" H 10150 2250 60  0001 C CNN
@@
 U 1 1 577B9ABD
 P 10150 2800
-F 0 "M5" H 10250 2800 40  0001 C CNN
+F 0 "M5" H 10150 2900 40  0000 C CNN
 F 1 "MOUNTING-HOLE" H 10150 2700 40  0001 C CNN
 F 2 "Mounting_Holes:MountingHole_2.5mm_Pad" H 10150 2550 60  0001 C CNN
@@
 	9300 3100 9550 3100
 $Comp
-L MOUNTING-HOLE M6
+L MOUNTING-HOLE M11
 U 1 1 577B9BA8
 P 10150 3100
-F 0 "M6" H 10250 3100 40  0001 C CNN
+F 0 "M11" H 10150 3200 40  0000 C CNN
 F 1 "MOUNTING-HOLE" H 10150 3000 40  0001 C CNN
 F 2 "Mounting_Holes:MountingHole_2.5mm_Pad" H 10150 2850 60  0001 C CNN
@@
 	9300 3400 9550 3400
 $Comp
-L MOUNTING-HOLE M7
+L MOUNTING-HOLE M12
 U 1 1 577B9BB7
 P 10150 3400
-F 0 "M7" H 10250 3400 40  0001 C CNN
+F 0 "M12" H 10150 3500 40  0000 C CNN
 F 1 "MOUNTING-HOLE" H 10150 3300 40  0001 C CNN
 F 2 "Mounting_Holes:MountingHole_2.5mm_Pad" H 10150 3150 60  0001 C CNN
@@
 	9300 3700 9550 3700
 $Comp
-L MOUNTING-HOLE M8
+L MOUNTING-HOLE M13
 U 1 1 577B9BC6
 P 10150 3700
-F 0 "M8" H 10250 3700 40  0001 C CNN
+F 0 "M13" H 10150 3800 40  0000 C CNN
 F 1 "MOUNTING-HOLE" H 10150 3600 40  0001 C CNN
 F 2 "Mounting_Holes:MountingHole_2.5mm_Pad" H 10150 3450 60  0001 C CNN
@@
 	9300 4000 9550 4000
 $Comp
-L MOUNTING-HOLE M9
+L MOUNTING-HOLE M17
 U 1 1 577B9BD5
 P 10150 4000
-F 0 "M9" H 10250 4000 40  0001 C CNN
+F 0 "M17" H 10150 4100 40  0000 C CNN
 F 1 "MOUNTING-HOLE" H 10150 3900 40  0001 C CNN
 F 2 "Mounting_Holes:MountingHole_2.5mm_Pad" H 10150 3750 60  0001 C CNN
@@
 	9300 4300 9550 4300
 $Comp
-L MOUNTING-HOLE M10
+L MOUNTING-HOLE M19
 U 1 1 577B9C8C
 P 10150 4300
-F 0 "M10" H 10250 4300 40  0001 C CNN
+F 0 "M19" H 10150 4400 40  0000 C CNN
 F 1 "MOUNTING-HOLE" H 10150 4200 40  0001 C CNN
 F 2 "Mounting_Holes:MountingHole_2.5mm_Pad" H 10150 4050 60  0001 C CNN
@@
 	9850 4300 10400 4300
 $Comp
-L MOUNTING-HOLE M1
+L MOUNTING-HOLE M28
 U 1 1 577BA5E6
 P 10150 1500
-F 0 "M1" H 10250 1500 40  0001 C CNN
+F 0 "M28" H 10150 1600 40  0000 C CNN
 F 1 "MOUNTING-HOLE" H 10150 1400 40  0001 C CNN
 F 2 "Mounting_Holes:MountingHole_2.5mm_Pad" H 10150 1250 60  0001 C CNN
@@
 	7600 1250 7600 1150
 $Comp
-L MOUNTING-HOLE M12
+L MOUNTING-HOLE M33
 U 1 1 577B70EB
 P 10950 1100
-F 0 "M12" H 11050 1100 40  0001 C CNN
+F 0 "M33" H 10950 1000 40  0000 C CNN
 F 1 "MOUNTING-HOLE" H 10950 1000 40  0001 C CNN
 F 2 "Mounting_Holes:MountingHole_2.5mm_Pad" H 10950 850 60  0001 C CNN
@@
 	10050 1100 10950 1100
 $Comp
-L MOUNTING-HOLE M13
+L MOUNTING-HOLE M0
 U 1 1 577B86A7
 P 10950 900
-F 0 "M13" H 11050 900 40  0001 C CNN
+F 0 "M0" H 10950 1000 40  0000 C CNN
 F 1 "MOUNTING-HOLE" H 10950 800 40  0001 C CNN
 F 2 "Mounting_Holes:MountingHole_2.5mm_Pad" H 10950 650 60  0001 C CNN
@@
 $EndComp
 $Comp
-L GND #PWR027
+L GND #PWR026
 U 1 1 5781F9CB
 P 11000 1500
-F 0 "#PWR027" H 11000 1250 50  0001 C CNN
+F 0 "#PWR026" H 11000 1250 50  0001 C CNN
 F 1 "GND" H 11000 1350 50  0000 C CNN
 F 2 "" H 11000 1500 50  0000 C CNN
@@
 $EndComp
 $Comp
-L GND #PWR028
+L GND #PWR027
 U 1 1 5781FDD2
 P 11000 1900
-F 0 "#PWR028" H 11000 1650 50  0001 C CNN
+F 0 "#PWR027" H 11000 1650 50  0001 C CNN
 F 1 "GND" H 11000 1750 50  0000 C CNN
 F 2 "" H 11000 1900 50  0000 C CNN
@@
 $EndComp
 $Comp
-L GND #PWR029
+L GND #PWR028
 U 1 1 5782227B
 P 11000 2200
-F 0 "#PWR029" H 11000 1950 50  0001 C CNN
+F 0 "#PWR028" H 11000 1950 50  0001 C CNN
 F 1 "GND" H 11000 2050 50  0000 C CNN
 F 2 "" H 11000 2200 50  0000 C CNN
@@
 $EndComp
 $Comp
-L GND #PWR030
+L GND #PWR029
 U 1 1 578222D9
 P 11000 2500
-F 0 "#PWR030" H 11000 2250 50  0001 C CNN
+F 0 "#PWR029" H 11000 2250 50  0001 C CNN
 F 1 "GND" H 11000 2350 50  0000 C CNN
 F 2 "" H 11000 2500 50  0000 C CNN
@@
 $EndComp
 $Comp
-L GND #PWR031
+L GND #PWR030
 U 1 1 578222DF
 P 11000 2800
-F 0 "#PWR031" H 11000 2550 50  0001 C CNN
+F 0 "#PWR030" H 11000 2550 50  0001 C CNN
 F 1 "GND" H 11000 2650 50  0000 C CNN
 F 2 "" H 11000 2800 50  0000 C CNN
@@
 $EndComp
 $Comp
-L GND #PWR032
+L GND #PWR031
 U 1 1 5782233D
 P 11000 3100
-F 0 "#PWR032" H 11000 2850 50  0001 C CNN
+F 0 "#PWR031" H 11000 2850 50  0001 C CNN
 F 1 "GND" H 11000 2950 50  0000 C CNN
 F 2 "" H 11000 3100 50  0000 C CNN
@@
 $EndComp
 $Comp
-L GND #PWR033
+L GND #PWR032
 U 1 1 57822343
 P 11000 3400
-F 0 "#PWR033" H 11000 3150 50  0001 C CNN
+F 0 "#PWR032" H 11000 3150 50  0001 C CNN
 F 1 "GND" H 11000 3250 50  0000 C CNN
 F 2 "" H 11000 3400 50  0000 C CNN
@@
 $EndComp
 $Comp
-L GND #PWR034
+L GND #PWR033
 U 1 1 57822349
 P 11000 3700
-F 0 "#PWR034" H 11000 3450 50  0001 C CNN
+F 0 "#PWR033" H 11000 3450 50  0001 C CNN
 F 1 "GND" H 11000 3550 50  0000 C CNN
 F 2 "" H 11000 3700 50  0000 C CNN
@@
 $EndComp
 $Comp
-L GND #PWR035
+L GND #PWR034
 U 1 1 5782234F
 P 11000 4000
-F 0 "#PWR035" H 11000 3750 50  0001 C CNN
+F 0 "#PWR034" H 11000 3750 50  0001 C CNN
 F 1 "GND" H 11000 3850 50  0000 C CNN
 F 2 "" H 11000 4000 50  0000 C CNN
@@
 $EndComp
 $Comp
-L GND #PWR036
+L GND #PWR035
 U 1 1 578223AD
 P 11000 4300
-F 0 "#PWR036" H 11000 4050 50  0001 C CNN
+F 0 "#PWR035" H 11000 4050 50  0001 C CNN
 F 1 "GND" H 11000 4150 50  0000 C CNN
 F 2 "" H 11000 4300 50  0000 C CNN
