File: hardware/name-blinker-2.kicad_pcb (KiCad board)
At the start: 2 copper layers, 70 x 50 mm, 40 parts, among them M1 MOUNTING-HOLE, M10 MOUNTING-HOLE, M12 MOUNTING-HOLE, M13 MOUNTING-HOLE, M2 MOUNTING-HOLE, M3 MOUNTING-HOLE, M4 MOUNTING-HOLE, M5 MOUNTING-HOLE, M6 MOUNTING-HOLE, M7 MOUNTING-HOLE, M8 MOUNTING-HOLE, M9 MOUNTING-HOLE, P1 CONN_01X08, P2 USB_OTG, SW2 SMD-TOGGLE-SWITCH-2CH_2X3P-7X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, U1 MCP73831, U2 BMD-300, U3 TPS63051

Commit message: add inductor
Parts:
- added C10: 1nF, Capacitors_SMD:C_0805_HandSoldering, F.Cu at (185.0, 105.1)
- added C7: 10uF, Capacitors_SMD:c_elec_4x5.8, F.Cu at (193.0, 105.5)
- added C8: 10uF, Capacitors_SMD:c_elec_4x5.8, F.Cu at (179.5, 109.0)
- added C9: 10uF, Capacitors_SMD:c_elec_4x5.8, F.Cu at (193.5, 110.0)
- added L1: LPS3015, lps3015:LPS3015, F.Cu at (187.0, 109.5)
- added R13: 1M, Resistors_SMD:R_0805_HandSoldering, F.Cu at (185.0, 105.1)
- added R14: 800K, Resistors_SMD:R_0805_HandSoldering, F.Cu at (185.0, 105.1)
- added R15: 2M, Resistors_SMD:R_0805_HandSoldering, F.Cu at (185.0, 105.1)
Connections:
- C3 pad 2: GND -> Net-(C3-Pad2)
- C6 pad 1: VCC -> +3V3
- M12 pad 1: VCC -> +3V3
- P1 pad 2: VCC -> +3V3
- P1 pad 4: GND -> UART_TX
- P1 pad 5: SWDIO -> UART_RX
- P1 pad 6: SWCLK -> SWDIO
- P1 pad 7: UART_TX -> SWCLK
- P1 pad 8: UART_RX -> GND
- U2 pad P17: VCC -> +3V3
- U3 pad P$10: Net-(U3-PadP$10) -> VCC
- U3 pad P$11: Net-(U3-PadP$11) -> VCC
- U3 pad P$12: Net-(U3-PadP$12) -> VCC
- U3 pad P$2: Net-(U3-PadP$2) -> GND
- U3 pad P$4: Net-(U3-PadP$4) -> +3V3
- U3 pad P$5: Net-(U3-PadP$5) -> +3V3
- U3 pad P$6: Net-(U3-PadP$6) -> GND
- U3 pad P$9: Net-(U3-PadP$9) -> GND

Commit message: some adjustments
Parts:
- P1: value CONN_01X08 -> CONN_01X09; footprint Pin_Headers:Pin_Header_Angled_1x08 -> Pin_Headers:Pin_Header_Angled_1x09
- moved P1 1.58 mm to (198.0, 55.5)
Connections:
- P1 pad 2: +3V3 -> VCC
- P1 pad 3: GND -> +3V3
- P1 pad 4: UART_TX -> GND
- P1 pad 5: UART_RX -> UART_TX
- P1 pad 6: SWDIO -> UART_RX
- P1 pad 7: SWCLK -> GND
- P1 pad 8: GND -> SWDIO

Commit message: charging circuit side
Parts:
- BT2: footprint Connectors_Molex:Molex_MicroLatch-53254-0270_02x2.00mm_Angled -> jst:Molex_MicroLatch-53254-0270_02x2.00mm_Angled
- U1: value MCP73831 -> (none)
- moved M12 64.0 mm to (153.0, 92.0)
- moved M1 63.5 mm to (217.0, 92.0)
- moved C8 47.8 mm to (168.5, 62.5)
- moved C9 47.3 mm to (182.5, 64.0)
- moved C10 46.6 mm to (175.5, 59.5)
- moved R14 43.7 mm to (163.5, 67.0)
- moved C7 41.2 mm to (169.0, 72.0)
- moved R15 40.9 mm to (170.0, 67.0)
- moved L1 39.9 mm to (176.5, 71.0)
- moved R13 35.1 mm to (184.5, 70.0)
- moved R12 18.7 mm to (207.5, 60.5), turned to 90 degrees
- moved D2 11.7 mm to (191.5, 64.0)
- moved R10 8.56 mm to (203.0, 60.5), turned to 180 degrees
- moved R11 8.50 mm to (195.0, 60.5), turned to 180 degrees
- moved U1 6.80 mm to (205.5, 65.0), turned to 0 degrees
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Connections:
- C3 pad 2: Net-(C3-Pad2) -> GND
- P1 pad 1: +5V -> SWCLK
- P1 pad 2: VCC -> SWDIO
- P1 pad 3: +3V3 -> GND
- P1 pad 4: GND -> UART_RX
- P1 pad 6: UART_RX -> GND
- P1 pad 7: GND -> +3V3
- P1 pad 8: SWDIO -> VCC
- P1 pad 9: SWCLK -> +5V
Routing:
- net Net-(BT1-Pad1): track 0.00 -> 72.6 mm
- net +5V: track 0.00 -> 31.0 mm, vias 0 -> 1
- net VCC: track 0.00 -> 17.6 mm, vias 0 -> 1
- net Net-(C3-Pad1): track 0.00 -> 16.3 mm
- net Net-(D1-Pad1): track 0.00 -> 12.9 mm
- net GND: track 0.00 -> 8.10 mm
- net Net-(D2-Pad2): track 0.00 -> 3.96 mm
- net Net-(D1-Pad2): track 0.00 -> 3.96 mm
- net Net-(R12-Pad1): track 0.00 -> 2.57 mm
- added copper zone on F.Cu, net GND
Other:
- net class Default: trace_width 0.25 -> 0.6

Commit message: connected all wires
Parts:
- removed C4, C5: 330pF, Capacitors_SMD:C_0805_HandSoldering
- added M11: MOUNTING-HOLE, Mounting_Holes:MountingHole_2.5mm_Pad, F.Cu at (203.0, 48.0)
- U1: value (none) -> MCP73831
- moved R15 17.7 mm to (176.5, 83.5), turned to 270 degrees
- moved C7 17.4 mm to (186.0, 68.5), turned to 270 degrees
- moved R14 17.0 mm to (176.5, 78.0), turned to 270 degrees
- moved R13 11.8 mm to (173.0, 72.5), turned to 180 degrees
- moved C10 11.0 mm to (178.8, 70.0)
- moved L1 11.0 mm to (181.0, 61.0)
- moved C6 8.60 mm to (170.0, 75.0), turned to 180 degrees
- moved C9 8.51 mm to (174.0, 63.5), turned to 90 degrees
- moved U3 3.64 mm to (179.0, 66.0), turned to 270 degrees
- moved C8 1.80 mm to (167.0, 63.5), turned to 90 degrees
Connections:
- P2 pad 2: Net-(P2-Pad2) -> (no net)
- P2 pad 3: Net-(P2-Pad3) -> (no net)
- P2 pad 4: Net-(P2-Pad4) -> (no net)
- SW2 pad CH1A: Net-(SW2-PadCH1A) -> (no net)
- SW2 pad CH1B: Net-(SW2-PadCH1B) -> (no net)
- SW2 pad CH2A: Net-(SW2-PadCH2A) -> (no net)
- SW2 pad COM1: Net-(SW2-PadCOM1) -> (no net)
- U2 pad P10: Net-(U2-PadP10) -> (no net)
- U2 pad P11: Net-(U2-PadP11) -> Net-(R14-Pad2)
- U2 pad P12: Net-(R14-Pad2) -> (no net)
- U2 pad P13: Net-(U2-PadP13) -> (no net)
- U2 pad P14: Net-(U2-PadP14) -> (no net)
- U2 pad P23: In0 -> (no net)
- U2 pad P25: Net-(C4-Pad1) -> (no net)
- U2 pad P26: Net-(C5-Pad1) -> (no net)
- U2 pad P32: Net-(U2-PadP32) -> (no net)
- U2 pad P33: Net-(U2-PadP33) -> (no net)
- U2 pad P34: Net-(U2-PadP34) -> (no net)
- U2 pad P36: Net-(U2-PadP36) -> (no net)
- U2 pad P38: Net-(U2-PadP38) -> (no net)
- U2 pad P39: Net-(U2-PadP39) -> (no net)
- U2 pad P40: Net-(U2-PadP40) -> (no net)
- U2 pad P41: Net-(U2-PadP41) -> (no net)
- U2 pad P42: Net-(U2-PadP42) -> (no net)
- U2 pad P6: Net-(U2-PadP6) -> (no net)
- U2 pad P7: Net-(U2-PadP7) -> (no net)
- U2 pad P8: Net-(U2-PadP8) -> (no net)
- U2 pad P9: Net-(U2-PadP9) -> In0
Routing:
- net +3V3: track 0.00 -> 119.0 mm, vias 0 -> 2
- net VCC: track 17.6 -> 80.8 mm, vias 1 -> 2
- net UART_TX: track 0.00 -> 62.8 mm, vias 0 -> 1
- net UART_RX: track 0.00 -> 59.8 mm, vias 0 -> 1
- net Out0: track 0.00 -> 59.7 mm, vias 0 -> 2
- net SWCLK: track 0.00 -> 54.6 mm, vias 0 -> 1
- net SWDIO: track 0.00 -> 53.1 mm, vias 0 -> 1
- net GND: track 8.10 -> 59.8 mm, vias 0 -> 6
- net In0: track 0.00 -> 50.5 mm, vias 0 -> 1
- net Out1: track 0.00 -> 48.8 mm, vias 0 -> 2
- net Out2: track 0.00 -> 46.9 mm, vias 0 -> 2
- net Out3: track 0.00 -> 39.5 mm, vias 0 -> 2
- net Out5: track 0.00 -> 32.5 mm, vias 0 -> 2
- net Out4: track 0.00 -> 31.0 mm
- net Out6: track 0.00 -> 20.3 mm
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Other:
- net class Default: trace_width 0.6 -> 0.25

Commit message: connected everything
Parts:
- added D10: LED, LEDs:LED_0805, F.Cu at (155.0, 76.0)
- added D11: LED, LEDs:LED_0805, F.Cu at (155.0, 84.0)
- added D3: LED, LEDs:LED_0805, F.Cu at (189.0, 50.0)
- added D4: LED, LEDs:LED_0805, F.Cu at (181.0, 50.0)
- added D5: LED, LEDs:LED_0805, F.Cu at (173.0, 50.0)
- added D6: LED, LEDs:LED_0805, F.Cu at (165.0, 50.0)
- added D7: LED, LEDs:LED_0805, F.Cu at (157.0, 50.0)
- added D8: LED, LEDs:LED_0805, F.Cu at (155.0, 60.0)
- added D9: LED, LEDs:LED_0805, F.Cu at (155.0, 68.0)
- added SW1: SW_PUSH, Buttons_Switches_SMD:SW_SPST_B3S-1000, F.Cu at (179.8, 91.2)
- moved R15 6.83 mm to (173.8, 77.2), turned to 90 degrees
- moved R5 1.00 mm to (161.0, 53.0)
- moved BT2 0.50 mm to (181.0, 88.5)
Connections:
- D2 pad 1: GND -> (no net)
Routing:
- net GND: track 59.8 -> 87.6 mm, vias 6 -> 11
- net Net-(BT1-Pad1): track 72.6 -> 63.9 mm
- net (no net): track 13.6 -> 6.00 mm, vias 2 -> 0
- net Net-(D3-Pad2): track 5.56 -> 12.0 mm
- net In0: track 50.5 -> 56.2 mm, vias 1 -> 0
- net Net-(D7-Pad2): track 5.14 -> 10.4 mm
- net Net-(D6-Pad2): track 5.56 -> 9.95 mm
- net Net-(D5-Pad2): track 5.56 -> 9.95 mm
- net Net-(D4-Pad2): track 5.56 -> 9.95 mm
- net Net-(D9-Pad2): track 5.56 -> 9.95 mm
- net Net-(D8-Pad2): track 5.14 -> 9.54 mm
- net Net-(D11-Pad2): track 5.97 -> 10.4 mm
- net Net-(D10-Pad2): track 5.97 -> 10.4 mm
- net Net-(R14-Pad2): track 7.92 -> 11.0 mm
- net Out5: track 32.5 -> 30.0 mm
Other:
- net class Default: trace_width 0.25 -> 0.6

Commit message: silkscreen stuff
Parts:
- removed M11: MOUNTING-HOLE, Mounting_Holes:MountingHole_2.5mm_Pad
Routing:
- net (no net): track 6.00 -> 3.00 mm
Other:
- board text added: "3V3"
- board text added: "5V"
- board text added: "Charge Complete"
- board text added: "Charging"
- board text added: "GND"
- board text added: "Name Blinker 2 Rev 1 (July 2016) Designer: Yeo Kheng Meng"
- board text added: "SWCLK"
- board text added: "SWDIO"
- board text added: "UART_RX"
- board text added: "UART_TX"
- board text added: "VCC"

Commit message: all lines connected
Parts:
- moved SW1 25.7 mm to (170.0, 67.5)
- moved C8 3.50 mm to (167.0, 60.0)
- moved C9 3.50 mm to (174.0, 60.0)
Routing:
- net In0: track 56.2 -> 79.5 mm, vias 0 -> 2
- net +3V3: track 119.0 -> 127.9 mm, vias 2 -> 1
- net SWCLK: track 54.6 -> 55.4 mm
- net GND: track 87.6 -> 87.0 mm
Other:
- net class Default: via_dia 0.6 -> 1
