File: hardware/name-blinker-2.kicad_pcb (KiCad board)
At the start: 2 copper layers, 70 x 50 mm, 56 parts, among them M1 MOUNTING-HOLE, M10 MOUNTING-HOLE, M12 MOUNTING-HOLE, M13 MOUNTING-HOLE, M2 MOUNTING-HOLE, M3 MOUNTING-HOLE, M4 MOUNTING-HOLE, M5 MOUNTING-HOLE, M6 MOUNTING-HOLE, M7 MOUNTING-HOLE, M8 MOUNTING-HOLE, M9 MOUNTING-HOLE, P1 CONN_01X09, P2 USB_OTG, SW1 SW_PUSH, SW2 SMD-TOGGLE-SWITCH-2CH_2X3P-7X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, U1 MCP73831, U2 BMD-300, U3 TPS63051

Commit message: final changes to rev 1
Parts:
- moved C7 6.90 mm to (185.9, 61.6)
Routing:
- net VCC: track 80.8 -> 85.9 mm
Other:
- net class Default: trace_width 0.6 -> 0.25
- board text added: "Off/On"
Changed lines of the file:
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@@
     (links 114)
     (no_connects 0)
-    (area 134.415477 28.915476 254.38316 99.475)
+    (area 149.924999 44.924999 220.075001 95.075001)
     (thickness 1.6)
-    (drawings 20)
-    (tracks 350)
+    (drawings 21)
+    (tracks 354)
     (zones 0)
     (modules 56)
@@
   )
   (setup
-    (last_trace_width 0.6)
+    (last_trace_width 0.25)
     (trace_clearance 0.2)
     (zone_clearance 0.508)
@@
   (net_class Default "This is the default net class."
     (clearance 0.2)
-    (trace_width 0.6)
+    (trace_width 0.25)
     (via_dia 1)
     (via_drill 0.4)
@@
     (at 181 61)
     (descr "LPS3015 Series")
-    (fp_text reference L1 (at -1.905 -1.905) (layer F.SilkS)
+    (fp_text reference L1 (at -0.8 -1.8) (layer F.SilkS)
       (effects (font (size 0.9652 0.9652) (thickness 0.18288)) (justify left bottom))
     )
-    (fp_text value LPS3015 (at 3.3 2.25 90) (layer F.SilkS)
+    (fp_text value LPS3015 (at -3 -3.3 180) (layer F.SilkS)
       (effects (font (size 0.77216 0.77216) (thickness 0.08128)) (justify left bottom))
     )
@@
     (tags "LED 0805 SMD")
     (attr smd)
-    (fp_text reference D2 (at -2.73 -0.06 90) (layer F.SilkS)
+    (fp_text reference D2 (at 2.7 0 90) (layer F.SilkS)
       (effects (font (size 1 1) (thickness 0.15)))
     )
@@
   )
   (module Capacitors_SMD:c_elec_4x5.8 (layer F.Cu)
-    (at 186 68.5 270)
+    (at 185.9 61.6 270)
     (descr "SMT capacitor, aluminium electrolytic, 4x5.8")
     (attr smd)
@@
       (effects (font (size 1 1) (thickness 0.15)))
     )
-    (fp_text value 10uF (at -4 0.5 360) (layer F.SilkS)
+    (fp_text value 10uF (at -4.1 0.1 360) (layer F.SilkS)
       (effects (font (size 1 1) (thickness 0.15)))
     )
@@
     (descr "Molex Micro-Latch connector, PN:53254-0270, side entry type, through hole")
     (tags "conn molex micro latch")
-    (fp_text reference BT2 (at 1.2 2.75 360) (layer F.SilkS)
+    (fp_text reference BT2 (at 3.6 2.7 360) (layer F.SilkS)
       (effects (font (size 1 1) (thickness 0.15)))
     )
@@
     (pad 2 smd rect (at 3.975 2.25 180) (size 1.55 1.3) (layers F.Cu F.Paste F.Mask)
       (net 2 GND))
+  )
+  (gr_text Off/On (at 218.9 81.7 90) (layer F.SilkS)
+    (effects (font (size 1.5 1.5) (thickness 0.3)))
   )
   (gr_arc (start 152 47) (end 150 47) (angle 90) (layer Edge.Cuts) (width 0.15))
@@
   (segment (start 193.65 60.5) (end 193.65 62.89902) (width 0.6) (layer F.Cu) (net 7))
   (segment (start 193.65 62.89902) (end 192.54902 64) (width 0.6) (layer F.Cu) (net 7))
+  (segment (start 180.149938 66.249938) (end 183.550062 66.249938) (width 0.25) (layer F.Cu) (net 8) (status 400000))
+  (segment (start 183.550062 66.249938) (end 185.9 63.9) (width 0.25) (layer F.Cu) (net 8) (status 800000))
+  (segment (start 185.9 63.9) (end 185.9 63.40086) (width 0.25) (layer F.Cu) (net 8) (status C00000))
+  (segment (start 179.749938 67.149938) (end 184.250062 67.149938) (width 0.25) (layer F.Cu) (net 8) (status 400000))
+  (segment (start 184.250062 67.149938) (end 185.9 65.5) (width 0.25) (layer F.Cu) (net 8))
+  (segment (start 180.149938 65.749937) (end 183.550923 65.749937) (width 0.25) (layer F.Cu) (net 8) (status 400000))
+  (segment (start 183.550923 65.749937) (end 185.9 63.40086) (width 0.25) (layer F.Cu) (net 8) (status 800000))
+  (segment (start 185.9 63.40086) (end 185.9 65.5) (width 1) (layer F.Cu) (net 8) (status 400000))
+  (segment (start 185.9 65.5) (end 185.9 70.40086) (width 1) (layer F.Cu) (net 8))
+  (segment (start 185.9 70.40086) (end 186 70.30086) (width 1) (layer F.Cu) (net 8))
   (segment (start 176.5 76.65) (end 179.65086 76.65) (width 1) (layer F.Cu) (net 8))
   (segment (start 179.65086 76.65) (end 186 70.30086) (width 1) (layer F.Cu) (net 8))
@@
   (segment (start 192.5 68) (end 203.9 68) (width 1) (layer F.Cu) (net 8))
   (segment (start 190.19914 70.30086) (end 192.5 68) (width 1) (layer F.Cu) (net 8))
-  (segment (start 179.749938 67.149938) (end 182.849078 67.149938) (width 0.25) (layer F.Cu) (net 8))
-  (segment (start 182.849078 67.149938) (end 186 70.30086) (width 0.25) (layer F.Cu) (net 8))
-  (segment (start 180.149938 65.749937) (end 181.449077 65.749937) (width 0.25) (layer F.Cu) (net 8))
-  (segment (start 181.449077 65.749937) (end 186 70.30086) (width 0.25) (layer F.Cu) (net 8))
-  (segment (start 180.149938 66.249938) (end 181.949078 66.249938) (width 0.25) (layer F.Cu) (net 8))
-  (segment (start 181.949078 66.249938) (end 186 70.30086) (width 0.25) (layer F.Cu) (net 8))
   (via (at 212.9 67) (size 0.6) (drill 0.4) (layers F.Cu B.Cu) (net 8))
   (segment (start 212.325 71.46) (end 212.3 67.3) (width 0.6) (layer F.Cu) (net 8))
