File: hardware/name-blinker-2.kicad_pcb (KiCad board)
At the start: 2 copper layers, 70 x 50 mm, 56 parts, among them M1 MOUNTING-HOLE, M10 MOUNTING-HOLE, M12 MOUNTING-HOLE, M13 MOUNTING-HOLE, M2 MOUNTING-HOLE, M3 MOUNTING-HOLE, M4 MOUNTING-HOLE, M5 MOUNTING-HOLE, M6 MOUNTING-HOLE, M7 MOUNTING-HOLE, M8 MOUNTING-HOLE, M9 MOUNTING-HOLE, P1 CONN_01X09, P2 USB_OTG, SW1 SW_PUSH, SW2 SMD-TOGGLE-SWITCH-2CH_2X3P-7X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, U1 MCP73831, U2 BMD-300, U3 TPS63051

Commit message: change mounting hole reference name to be in line with connected NRF pins
Parts:
- renumbered M13 to M0, M6 to M11, M7 to M12, M8 to M13, M9 to M17, M10 to M19, M1 to M28, M12 to M33
Connections:
- P2 pad 2: Net-(P2-Pad2) -> (no net)
- P2 pad 3: Net-(P2-Pad3) -> (no net)
- P2 pad 4: Net-(P2-Pad4) -> (no net)
- SW2 pad CH1A: Net-(SW2-PadCH1A) -> (no net)
- SW2 pad CH1B: Net-(SW2-PadCH1B) -> (no net)
- SW2 pad CH2A: Net-(SW2-PadCH2A) -> (no net)
- SW2 pad COM1: Net-(SW2-PadCOM1) -> (no net)
- U2 pad P10: Net-(U2-PadP10) -> (no net)
- U2 pad P12: Net-(U2-PadP12) -> (no net)
- U2 pad P13: Net-(U2-PadP13) -> (no net)
- U2 pad P14: Net-(U2-PadP14) -> (no net)
- U2 pad P23: Net-(U2-PadP23) -> (no net)
- U2 pad P25: Net-(U2-PadP25) -> (no net)
- U2 pad P26: Net-(U2-PadP26) -> (no net)
- U2 pad P32: Net-(U2-PadP32) -> (no net)
- U2 pad P33: Net-(U2-PadP33) -> (no net)
- U2 pad P34: Net-(U2-PadP34) -> (no net)
- U2 pad P36: Net-(U2-PadP36) -> (no net)
- U2 pad P38: Net-(U2-PadP38) -> (no net)
- U2 pad P39: Net-(U2-PadP39) -> (no net)
- U2 pad P40: Net-(U2-PadP40) -> (no net)
- U2 pad P41: Net-(U2-PadP41) -> (no net)
- U2 pad P42: Net-(U2-PadP42) -> (no net)
- U2 pad P6: Net-(U2-PadP6) -> (no net)
- U2 pad P7: Net-(U2-PadP7) -> (no net)
- U2 pad P8: Net-(U2-PadP8) -> (no net)
